File: full.brd (EAGLE design)
At the start: 100 x 80 mm, 19 parts, among them T1 2SC1815, T2 2SC1815, T3 2SC1815

Commit message: スイッチ追加
Parts:
- added S1: 9077-2, switch-misc:9077-2
Connections:
- new net N$14: B1.P29
- net GND: now also S1.3
- net N$29: now also S1.1
Changed lines of the file:
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@@
 <element name="R7" library="rcl" package="0204/7" value="10k" x="66.04" y="13.97" rot="R90"/>
 <element name="JP5" library="pinhead" package="1X03" value="" x="2.54" y="15.24" rot="R270"/>
+<element name="S1" library="switch-misc" package="9077-2" value="9077-2" x="-7.62" y="7.62"/>
 </elements>
 <signals>
@@
 <wire x1="96.52" y1="7.62" x2="45.72" y2="7.62" width="0.4064" layer="16"/>
 <wire x1="45.72" y1="7.62" x2="45.72" y2="20.32" width="0.4064" layer="16"/>
+<contactref element="S1" pad="3"/>
+<wire x1="-5.08" y1="10.16" x2="2.54" y2="15.24" width="0" layer="19" extent="1-1"/>
 </signal>
 <signal name="N$7">
@@
 <via x="66.04" y="63.5" extent="1-16" drill="0.6" shape="square"/>
 <wire x1="66.04" y1="63.5" x2="66.04" y2="17.78" width="0.4064" layer="16"/>
+<contactref element="S1" pad="1"/>
+<wire x1="-10.16" y1="10.16" x2="66.04" y2="17.78" width="0" layer="19" extent="1-1"/>
 </signal>
 <signal name="VBUS">
@@
 <contactref element="B1" pad="VU"/>
 </signal>
+<signal name="N$14">
+<contactref element="B1" pad="P29"/>
+</signal>
 </signals>
