File: full.sch (EAGLE design)
At the start: 19 parts, among them T1 2SC1815, T2 2SC1815, T3 2SC1815

Commit message: スイッチ追加
Parts:
- added S1: 9077-2, switch-misc:9077-2
Connections:
- new net N$14: B1.P29
- net GND: now also S11.O
- net N$29: now also S11.S
Changed lines of the file:
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@@
 <part name="JP5" library="pinhead" deviceset="PINHD-1X3" device=""/>
 <part name="SUPPLY17" library="supply2" deviceset="+5V" device=""/>
+<part name="S1" library="switch-misc" deviceset="9077-2" device=""/>
+<part name="SUPPLY18" library="supply2" deviceset="GND" device=""/>
 </parts>
 <sheets>
@@
 <instance part="JP5" gate="A" x="35.56" y="15.24"/>
 <instance part="SUPPLY17" gate="+5V" x="12.7" y="15.24"/>
+<instance part="S1" gate="1" x="-20.32" y="20.32" rot="R180"/>
+<instance part="S1" gate="2" x="-10.16" y="20.32" rot="R180"/>
+<instance part="SUPPLY18" gate="GND" x="-17.78" y="12.7"/>
 </instances>
 <busses>
@@
 <pinref part="SUPPLY12" gate="GND" pin="GND"/>
 <wire x1="33.02" y1="15.24" x2="17.78" y2="15.24" width="0.1524" layer="91"/>
+</segment>
+<segment>
+<pinref part="S1" gate="1" pin="O"/>
+<pinref part="SUPPLY18" gate="GND" pin="GND"/>
 </segment>
 </net>
@@
 <wire x1="-20.32" y1="96.52" x2="68.58" y2="96.52" width="0.1524" layer="91"/>
 <wire x1="68.58" y1="96.52" x2="68.58" y2="43.18" width="0.1524" layer="91"/>
-</segment>
-</net>
+<wire x1="-20.32" y1="86.36" x2="-27.94" y2="86.36" width="0.1524" layer="91"/>
+<wire x1="-27.94" y1="86.36" x2="-27.94" y2="15.24" width="0.1524" layer="91"/>
+<pinref part="S1" gate="1" pin="S"/>
+<wire x1="-27.94" y1="15.24" x2="-22.86" y2="15.24" width="0.1524" layer="91"/>
+</segment>
+</net>
+<net name="N$14" class="0">
+<segment>
+<pinref part="B1" gate="G$1" pin="P29"/>
+<wire x1="-15.24" y1="58.42" x2="-20.32" y2="58.42" width="0.1524" layer="91"/>
+<wire x1="-20.32" y1="58.42" x2="-20.32" y2="25.4" width="0.1524" layer="91"/>
+</segment>
+</net>
